File: Circuit Schematics/Kicad Files/Car_Circuit.kicad_sch (KiCad schematic)
At the start: 10 parts

Commit message: Update Schematic
Fixed a mistake in Schematic
Parts:
- A: value (none) -> Arduino_Nano; footprint (none) -> Module:Arduino_Nano
- BT1: value (none) -> Battery
- M1, M2: value (none) -> Motor_DC
- SW1: value (none) -> SW_SPST
- U1: value (none) -> bq24074
- U2: value (none) -> LC709203F
- U3: value (none) -> U1V11F5
- U4: value (none) -> DRV8833
- U5: value (none) -> NRF24L01; footprint (none) -> RF_Module:nRF24L01_Breakout
Connections:
- net at U4.13 (BIN2): now also A.6 (D3); no longer A.8 (D5)
- net at U4.15 (AIN2): now also A.8 (D5); no longer A.6 (D3)
- net at U4.16 (AIN1): now also A.9 (D6); no longer A.5 (D2)
- net at U5.3 (CE): now also A.13 (D10); no longer A.10 (D7)
- net at U5.4 (~{CSN}): now also A.5 (D2); no longer A.11 (D8)
